Commit message: hh

File: urdf/aws_amr_description.urdf (robot description, URDF)
Before this commit: robot aws_amr_description, 10 links, 9 joints
Links:
- link FL_steering_link: mass 0.21503 -> 0.215025529188031
- link FL_wheel: mass 0.95802 -> 0.958024018560995
- link FR_steering_link: mass 0.21503 -> 0.21502552911799
- link FR_wheel: mass 0.95802 -> 0.958024049096675
- link RL_steering_link: mass 0.21503 -> 0.215025508213933
- link RL_wheel: mass 0.95802 -> 0.95802404699446
- link RR_steering_link: mass 0.21503 -> 0.215025525294734
- link RR_wheel: mass 0.95802 -> 0.958024083703301
- link basefootprint_link: mass 0 -> 40.12833
Joints:
- joint FL_steering_joint: origin xyz=0.24162 -0.2879 0.1095 rpy=0 0 0 -> xyz=0.241621591099171 -0.287902443050945 0.1095 rpy=0 0 0
- joint base_joint: origin xyz=0.00089997 0 0.089894 rpy=0 0 0 -> xyz=0.000899965730756125 0 0.0898937183015765 rpy=0 0 0
